File: SprinklerControllerSTM.kicad_pcb (KiCad board)
At the start: 2 copper layers, 200 x 110 mm, 434 parts, among them J1 USB_B_Micro, J10 Conn_01x02, J11 Conn_01x04, J12 Conn_01x06, J13 Conn_01x05, J14 Conn_01x01, J16 Conn_01x02, J17 Conn_01x02, J18 Conn_01x02, J2 Screw_Terminal_01x10, J20 Conn_01x06, J21 Conn_01x04, J22 Conn_01x06, J23 Conn_01x04, J25 Conn_01x06, J26 Conn_01x02, J27 Conn_01x03, J28 Conn_01x03, J29 Micro_SD_Card_Det_Hirose_DM3AT, J3 Screw_Terminal_01x10, J30 USB_B_Micro, J4 Screw_Terminal_01x10, J5 Screw_Terminal_01x10, J6 Screw_Terminal_01x10, J7 Screw_Terminal_01x02, J8 Conn_01x02, J9 Conn_01x03, SW1 SW_Push, SW2 SW_Push, SW3 SW_Push, SW4 SW_Push, U1 STM32F078VBTx, U10 MOC3012M, U11 MOC3012M, U12 LT1117-3.3, U13 MOC3012M, U14 MOC3012M, U15 MOC3012M, U16 MOC3012M, U17 MOC3012M, U18 MOC3012M, U19 MOC3012M, U2 NCP1117-1.8_SOT223, U20 MOC3012M, U21 mcp6s93, U22 MOC3012M, U23 MOC3012M, U24 MOC3012M, U25 MOC3012M, U26 MOC3012M, U27 MOC3012M, U28 MOC3012M, U29 MOC3012M, U3 ACS723xLCTR-05AB, U30 MCP6G03, U31 MOC3012M, U32 MOC3012M, U33 MOC3012M, U34 MOC3012M, U35 MOC3012M, U36 MOC3012M, U37 MOC3012M, U38 MOC3012M, U39 FT234XD, U4 MOC3012M, U40 MOC3012M, U41 MOC3012M, U42 MOC3012M, U43 MOC3012M, U44 MOC3012M, U45 MOC3012M, U46 MOC3012M, U47 MOC3012M, U48 MC34063AD, U5 MOC3012M, U6 MOC3012M, U7 MOC3012M, U8 MOC3012M, U9 MOC3012M, Y1 16Mhz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

Commit message: add some files
Parts:
- C77: value 18pf -> 0.1uf
- R100, R103, R106, R109, R112, R115, R118, R12, R121, R124, R127, R130, R133, R136, R139, R142, R145, R148, R15, R151, R154, R157, R160, R163, R164, R165, R166, R167, R168, R17, R18, R19, R20, R21, R22, R23, R24, R25, R26, R28, R31, R34, R35, R36, R37, R38, R39, R40, R41, R42, R45, R48, R51, R52, R53, R54, R55, R56, R57, R58, R59, R62, R65, R67, R68, R69, R70, R71, R72, R73, R74, R76, R79, R82, R85, R88, R9, R91, R94, R97: value 510 -> 220
