File: optodriver.sch (KiCad schematic (older format))
At the start: 8 parts, among them U4 MOC3012M

Commit message: add some files
Parts:
- R17, R9: value 510 -> 220
Changed lines of the file:
@@
 AR Path="/5BF4B528/5BFB147C/5BF8D198" Ref="R160"  Part="1"
 F 0 "R9" H 4770 2896 50  0000 L CNN
-F 1 "510" H 4770 2805 50  0000 L CNN
+F 1 "220" H 4770 2805 50  0000 L CNN
 F 2 "Resistor_SMD:R_0603_1608Metric" V 4630 2850 50  0001 C CNN
 F 3 "~" H 4700 2850 50  0001 C CNN
@@
 AR Path="/5BF4B528/5BFB147C/5C1BEF98" Ref="R56"  Part="1"
 F 0 "R17" H 4470 2646 50  0000 L CNN
-F 1 "510" H 4470 2555 50  0000 L CNN
+F 1 "220" H 4470 2555 50  0000 L CNN
 F 2 "Resistor_SMD:R_0603_1608Metric" V 4330 2600 50  0001 C CNN
 F 3 "~" H 4400 2600 50  0001 C CNN
